File: Test-Signal-Generator/Test-Signal-Generator.sch (KiCad schematic (older format))
At the start: 18 parts, among them J1 AudioJack3, U1 MCP6002-xP

Commit message: Finished schematic & added notes
Parts:
- added C6, C8: 100nF, symbol Device:C_Small
- added C7: 1uF, symbol Device:C_Small
- added C9: 100uF, symbol Device:CP1_Small
- added D4: LED, symbol Device:LED
- added R10, R9: 10k, symbol Device:R
- added R11, R12: 150, symbol Device:R
- added R13: 470, symbol Device:R
- added R8: 180k, symbol Device:R
- added RV1: R_POT, symbol Device:R_POT
- added SW1: SW_Push_SPDT, symbol Switch:SW_Push_SPDT
- added U2: MCP6002-xP, symbol Amplifier_Operational:MCP6002-xP
- gave numbers to parts that had none: 2
Connections:
- net GND: now also Batt_3V.2 (-), D1.2 (A), J1.S, C8.2, C9.2, D4.1 (K), U2.4 (V-)
- net Vcc: now also C8.1, C9.1, R13.2, SW1.2 (B), U2.8 (V+)
- net at C5.1, D2.1 (K), D3.2 (A)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: now also R9.1, RV1.3, U2.5 (+)
- net at R7.2, U1.6 (-): now also C6.2, R8.1
- net at U1.7: now also C6.1, C7.2, R8.2
- net at Batt_3V.1 (+): now also D1.1 (K), SW1.3 (C)
- net at J1.R: now also R12.2
- net at J1.T: now also R11.2
- new net: D4.2 (A), R13.1
- new net: R10.2, R11.1, U2.1
- new net: R10.1, R9.2, U2.2 (-)
- new net: RV1.2, U2.3 (+)
- new net: R12.1, U2.6 (-), U2.7
- new net: C7.1, RV1.1
Other:
- note added: "Switch is controlled via\naudio jack"
- note added: "f = 1/(sqrt(6) * 2pi * R1,2,3 * C1,2,3)"
- moved on the sheet: Batt_3V, D1, J1
